File: schematics/Tachoconverter.kicad_sch (KiCad schematic)
At the start: 30 parts, among them J1 Motor, J2 HC05, J3 Input, J4 Conn_01x01, J5 Conn_01x02, J6 Conn_01x07, J7 Conn_01x01, J8 Conn_01x07, J9 Conn_01x01, U1 AT24CS64-SSHM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

Commit message: board changed
Parts:
- removed J8: Conn_01x07, Connector_PinHeader_2.54mm:PinHeader_1x07_P2.54mm_Vertical, symbol Connector_Generic:Conn_01x07
- removed U3: 74LVC2GU04, Package_TO_SOT_SMD:SOT-23-6_Handsoldering, symbol 74xGxx:74LVC2GU04
- added J10: Conn_01x05, Connector_PinHeader_2.54mm:PinHeader_1x05_P2.54mm_Vertical, symbol Connector_Generic:Conn_01x05
- added J8: Conn_01x01, Connector_PinHeader_2.54mm:PinHeader_1x01_P2.54mm_Vertical, symbol Connector_Generic:Conn_01x01
- added R5, R6: 1k, Resistor_SMD:R_1206_3216Metric_Pad1.30x1.75mm_HandSolder, symbol Device:R_Small
- added U5: 74HC14, Package_SO:SOIC-14_3.9x8.7mm_P1.27mm, symbol 74xx:74HC14
Connections:
- net +3V3: now also R5.1, R6.1; no longer R4.1
- net +5V: now also R4.1, U5.14 (VCC); no longer J2.5 (Pin_5)
- net GND: now also U5.7 (GND)
- net MotorPWM: now also U5.5
- net MotorSpeed: now also U5.4; no longer J1.2 (Pin_2), R4.2
- net SCL: now also R6.2
- net SDA: now also R5.2
- net VSpeedIn: now also A1.27 (D5/MISO1), U5.2; no longer A1.22 (D0/SDA2)
- net at J1.5 (Pin_5): now also U5.6
- net at A1.23 (D1/SCL2): now also J10.2 (Pin_2)
- net at A1.24 (D2): now also J10.3 (Pin_3)
- net at A1.25 (D3): now also J10.4 (Pin_4)
- net at A1.26 (D4/MOSI1): now also J10.5 (Pin_5)
- net at A1.29 (D7/SS1): now also J8.1 (Pin_1)
- net at J7.1 (Pin_1): now also A1.33 (D11); no longer A1.32 (D10)
- net at D2.3 (K), R3.2: now also U5.1
- new net: J1.2 (Pin_2), R4.2, U5.3
- new net: A1.22 (D0/SDA2), J10.1 (Pin_1)
- new net: J2.5 (Pin_5), U5.10, U5.12, U5.8
- new net ~{HC05ON}: A1.32 (D10), U5.11, U5.13, U5.9
Other:
- moved on the sheet: J7, R2

Commit message: schematic update
Parts:
- H1, H2, H3, H4: footprint MountingHole:MountingHole_2.7mm_M2.5 -> MountingHole:MountingHole_3.2mm_M3
Connections:
- net SCL: now also A1.5 (SDA1/D16), R5.2; no longer A1.4 (SCL1/D15), R6.2
- net SDA: now also A1.4 (SCL1/D15), R6.2; no longer A1.5 (SDA1/D16), R5.2
Other:
- note added: "Symbol Wrong! D15=SDA D16=SCL"
- moved on the sheet: R5, R6
